File: projeto/_autosave-lhc_tijolo32_board.kicad_pcb (KiCad board)
At the start: 2 copper layers, 25.4 x 59.2 mm, 28 parts, among them J1 USB_C_Receptacle_USB2.0, J2 Conn_01x04_Female, Q1 MMBT3904, Q2 MMBT3904, SW1 SW_Push, SW2 SW_Push, U1 TLV75733PDBV, U2 CH340G, U3 ESP32-WROOM-32D, Y1 Crystal_GND24_Small

Commit message: Schematic update
Parts:
- added G***: LOGO, lhc_logos:tijolo32_medium_mask, B.Cu at (123.4, 101.3)
- G***: moved to B.Cu
- moved G*** 48.7 mm to (123.4, 101.3), turned to 180 degrees
