File: projeto/_autosave-lhc_tijolo32_board.sch (KiCad schematic (older format))
At the start: 46 parts, among them J1 USB_C_Receptacle_USB2.0, J2 OLED, J3 JTAG 10pin Connector, Q1 MMBT3904, Q2 MMBT3904, SW1 SW_Push, SW2 SW_Push, U1 AMS1117-3.3, U2 CH340G, U3 ESP32-WROOM-32D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

Commit message: Schematic update
Connections:
- net +3V3: now also B1.19 (37)
- net GND: now also B1.18 (38)
- no-connect marks 9 -> 7
Changed lines of the file:
@@
 	0    1    1    0
 $EndComp
-NoConn ~ 9450 1950
-NoConn ~ 9450 1850
 Text GLabel 9350 1750 0    50   Input ~ 0
 SVP
@@
 Wire Wire Line
 	950  7250 1250 7250
+$Comp
+L power:+3V3 #PWR?
+U 1 1 5F90819A
+P 9050 1750
+F 0 "#PWR?" H 9050 1600 50  0001 C CNN
+F 1 "+3V3" H 9050 1900 50  0000 C CNN
+F 2 "" H 9050 1750 50  0001 C CNN
+F 3 "" H 9050 1750 50  0001 C CNN
+	1    9050 1750
+	1    0    0    -1
+$EndComp
+$Comp
+L power:GND #PWR?
+U 1 1 5F908A0D
+P 9000 1950
+F 0 "#PWR?" H 9000 1700 50  0001 C CNN
+F 1 "GND" V 9000 1750 50  0000 C CNN
+F 2 "" H 9000 1950 50  0001 C CNN
+F 3 "" H 9000 1950 50  0001 C CNN
+	1    9000 1950
+	0    1    1    0
+$EndComp
+Wire Wire Line
+	9050 1750 9050 1850
+Wire Wire Line
+	9050 1850 9450 1850
+Wire Wire Line
+	9000 1950 9450 1950
 $EndSCHEMATC
