File: projeto/lhc_tijolo32_board.kicad_pcb (KiCad board)
At the start: 2 copper layers, 25.4 x 59.2 mm, 28 parts, among them J1 USB_C_Receptacle_USB2.0, J2 Conn_01x04_Female, Q1 MMBT3904, Q2 MMBT3904, SW1 SW_Push, SW2 SW_Push, U1 TLV75733PDBV, U2 CH340G, U3 ESP32-WROOM-32D, Y1 Crystal_GND24_Small

Commit message: Schematic update
Parts:
- removed B1: ESP32_THING_W_ANT_KEEPOUT, Boards:ESP32_THING
- removed C1, C2, C3, C4, C5, C6, C7, C8: C_Small, Capacitor_SMD:C_0603_1608Metric
- removed D1: LED, LED_SMD:LED_0805_2012Metric
- removed G***: LOGO, lhc_logos:tijolo32_medium_cu
- removed G***: LOGO, lhc_logos:brick_wall_medium
- removed G***: LOGO, lhc_logos:lhc_logo_alt_xlarge
- removed J1: USB_C_Receptacle_USB2.0, Connector_USB:USB_C_Receptacle_Palconn_UTC16-G
- removed J2: Conn_01x04_Female, Connector_PinHeader_2.54mm:PinHeader_1x04_P2.54mm_Vertical
- removed Q1, Q2: MMBT3904, Package_TO_SOT_SMD:SOT-23
- removed R1, R4, R5: 10kR, Resistor_SMD:R_0603_1608Metric
- removed R2, R3: 5k1R, Resistor_SMD:R_0603_1608Metric
- removed SW1, SW2: SW_Push, Switches:TACTILE_SWITCH_SMD_6.0X3.5MM
- removed U1: TLV75733PDBV, Package_TO_SOT_SMD:SOT-23-5
- removed U2: CH340G, Package_SO:SOIC-16_3.9x9.9mm_P1.27mm
- removed U3: ESP32-WROOM-32D, RF_Module:ESP32-WROOM-32
- removed Y1: Crystal_GND24_Small, Crystal:Crystal_SMD_EuroQuartz_MT-4Pin_3.2x2.5mm
Other:
- board outline removed
- net class Default: clearance 0.127 -> 0.2; trace_width 0.127 -> 0.25; via_dia 0.6 -> 0.8; via_drill 0.3 -> 0.4
- rule pad_to_mask_clearance: 0.051 -> 0
- rule trace_clearance: 0.127 -> 0.2
- rule trace_min: 0.127 -> 0.2
- rule via_min_size: 0.6 -> 0.4

Commit message: Schematic update
Parts:
- added B1: ESP32_THING_W_ANT_KEEPOUT, Boards:ESP32_THING, F.Cu at (101.6, 110.5)
- added C1: 1uF, Capacitor_SMD:C_0603_1608Metric, F.Cu at (133.1, 102.2)
- added C10: 10uF, Capacitor_Tantalum_SMD:CP_EIA-3216-12_Kemet-S, F.Cu at (164.2, 59.9)
- added C11: 10nF, Capacitor_SMD:C_0603_1608Metric, F.Cu at (182.2, 54.7)
- added C12: 100nF, Capacitor_SMD:C_0603_1608Metric, F.Cu at (164.2, 41.1)
- added C13: 100nF, Capacitor_SMD:C_0603_1608Metric, F.Cu at (178.2, 54.9)
- added C14: 100nF, Capacitor_SMD:C_0603_1608Metric, F.Cu at (197.6, 66.2)
- added C15: ?pF, Capacitor_SMD:C_0603_1608Metric, F.Cu at (167.1, 64.1)
- added C16: ?pF, Capacitor_SMD:C_0603_1608Metric, F.Cu at (173.4, 59.3)
- added C2: 100nF, Capacitor_SMD:C_0603_1608Metric, F.Cu at (129.1, 107.3)
- added C3: ?pF, Capacitor_SMD:C_0603_1608Metric, F.Cu at (129.3, 98.7)
- added C4: ?pF, Capacitor_SMD:C_0603_1608Metric, F.Cu at (132.2, 97.7)
- added C5: 1uF, Capacitor_SMD:C_0603_1608Metric, F.Cu at (167.1, 69.1)
- added C6: 100nF, Capacitor_SMD:C_0603_1608Metric, F.Cu at (167.1, 66.6)
- added C7: 100nF, Capacitor_SMD:C_0603_1608Metric, F.Cu at (171.1, 64.1)
- added C8: 100nF, Capacitor_SMD:C_0603_1608Metric, F.Cu at (138.7, 93.8)
- added C9: 100nF, Capacitor_SMD:C_0603_1608Metric, F.Cu at (106.9, 88.4)
- added D1: LED, LED_SMD:LED_0805_2012Metric, F.Cu at (117.5, 82.7)
- added F1: 1A PTC, Resistor_SMD:R_1210_3225Metric, F.Cu at (118.0, 100.6)
- added G***: LOGO, lhc_logos:tijolo32_medium_mask, B.Cu at (114.2, 53.1)
- added G***: LOGO, lhc_logos:tijolo32_medium_cu, B.Cu at (114.2, 53.0)
- added J1: USB_C_Receptacle_USB2.0, Connector_USB:USB_C_Receptacle_Palconn_UTC16-G, B.Cu at (114.2, 106.0)
- added J2: OLED, Connector_PinHeader_2.54mm:PinHeader_1x04_P2.54mm_Vertical, F.Cu at (110.6, 75.2)
- added J3: JTAG 10pin Connector, Connector_PinHeader_1.27mm:PinHeader_2x05_P1.27mm_Vertical_SMD, B.Cu at (114.9, 94.6)
- added J4: Conn_01x20_Male, Connector_PinHeader_2.54mm:PinHeader_1x20_P2.54mm_Vertical, B.Cu at (102.9, 109.2)
- added JP1: P2, Jumper:SolderJumper-3_P1.3mm_Bridged12_Pad1.0x1.5mm_NumberLabels, B.Cu at (114.3, 78.7)
- added JP2: P1, Jumper:SolderJumper-3_P1.3mm_Bridged12_Pad1.0x1.5mm_NumberLabels, B.Cu at (109.5, 78.7)
- added Q1: MMBT3904, Package_TO_SOT_SMD:SOT-23, F.Cu at (120.8, 87.5)
- added Q2: MMBT3904, Package_TO_SOT_SMD:SOT-23, F.Cu at (169.2, 60.6)
- added R1: 10kR, Resistor_SMD:R_0603_1608Metric, F.Cu at (121.0, 78.7)
- added R10: 0R, Resistor_SMD:R_0603_1608Metric, F.Cu at (114.9, 103.9)
- added R11: 0R, Resistor_SMD:R_0603_1608Metric, F.Cu at (113.2, 103.9)
- added R12: 0R, Resistor_SMD:R_0603_1608Metric, F.Cu at (106.5, 98.8)
- added R13: 0R, Resistor_SMD:R_0603_1608Metric, F.Cu at (197.6, 68.7)
- added R2: 5k1R, Resistor_SMD:R_0603_1608Metric, F.Cu at (116.5, 106.8)
- added R3: 5k1R, Resistor_SMD:R_0603_1608Metric, F.Cu at (111.9, 106.8)
- added R4: 10kR, Resistor_SMD:R_0603_1608Metric, F.Cu at (158.6, 79.2)
- added R5: 10kR, Resistor_SMD:R_0603_1608Metric, F.Cu at (178.2, 57.4)
- added R6: 10kR, Resistor_SMD:R_0603_1608Metric, F.Cu at (138.7, 96.3)
- added R7: 1kR, Resistor_SMD:R_0603_1608Metric, F.Cu at (183.8, 51.3)
- added R8: 10kR, Resistor_SMD:R_0603_1608Metric, F.Cu at (164.3, 75.0)
- added R9: 10kR, Resistor_SMD:R_0603_1608Metric, F.Cu at (187.9, 51.3)
- added SW1: SW_Push, Switches:TACTILE_SWITCH_SMD_6.0X3.5MM, F.Cu at (106.4, 104.9)
- added SW2: SW_Push, Switches:TACTILE_SWITCH_SMD_6.0X3.5MM, F.Cu at (122.0, 104.9)
- added U1: AMS1117-3.3, Package_TO_SOT_SMD:SOT-223-3_TabPin2, F.Cu at (110.2, 81.4)
- added U2: CH340G, Package_SO:SOIC-16_3.9x9.9mm_P1.27mm, F.Cu at (110.5, 93.5)
- added U3: ESP32-WROOM-32D, RF_Module:ESP32-WROOM-32, F.Cu at (114.3, 62.4)
- added Y1: 12MHz 10ppm, Crystal:Crystal_SMD_EuroQuartz_MT-4Pin_3.2x2.5mm, F.Cu at (131.4, 93.3)
- added Y2: 32k 20ppm, Crystal:Crystal_SMD_3215-2Pin_3.2x1.5mm, F.Cu at (179.3, 51.7)
Routing:
- net Net-(F1-Pad2): track 0.00 -> 10.5 mm, vias 0 -> 1
- net D-: track 0.00 -> 8.54 mm
- net D+: track 0.00 -> 8.54 mm
- net Net-(J1-PadA7): track 0.00 -> 6.75 mm, vias 0 -> 1
- net Net-(J1-PadA6): track 0.00 -> 6.10 mm, vias 0 -> 1
- net Net-(J1-PadA5): track 0.00 -> 2.93 mm, vias 0 -> 1
- net GND: track 0.00 -> 2.72 mm
- net Net-(J1-PadB5): track 0.00 -> 2.71 mm, vias 0 -> 1
- added copper zone on F.Cu, net GND
Other:
- board outline added: 25.4 x 64.8 mm
- net class Default: clearance 0.2 -> 0.127; trace_width 0.25 -> 0.127; via_dia 0.8 -> 0.6; via_drill 0.4 -> 0.3
- rule pad_to_mask_clearance: 0 -> 0.051
- rule trace_clearance: 0.2 -> 0.127
- rule trace_min: 0.2 -> 0.127
- rule via_min_size: 0.4 -> 0.6
