File: projeto/lhc_tijolo32_board.sch (KiCad schematic (older format))
At the start: 46 parts, among them J1 USB_C_Receptacle_USB2.0, J2 OLED, J3 JTAG 10pin Connector, Q1 MMBT3904, Q2 MMBT3904, SW1 SW_Push, SW2 SW_Push, U1 AMS1117-3.3, U2 CH340G, U3 ESP32-WROOM-32D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

Commit message: Schematic update
Parts:
- C15, C16, C3, C4: value 20pF -> ?pF
- Y2: footprint (none) -> Crystal:Crystal_SMD_3215-2Pin_3.2x1.5mm
Connections:
- net +3V3: now also B1.19 (37)
- net GND: now also B1.18 (38)
- no-connect marks 9 -> 7
Changed lines of the file:
@@
 P 2700 7150
 F 0 "C3" H 2800 7150 50  0000 L CNN
-F 1 "20pF" H 2750 7050 50  0000 L CNN
+F 1 "?pF" H 2800 7050 50  0000 L CNN
 F 2 "Capacitor_SMD:C_0603_1608Metric" H 2700 7150 50  0001 C CNN
 F 3 "~" H 2700 7150 50  0001 C CNN
@@
 P 2200 7150
 F 0 "C4" H 2300 7150 50  0000 L CNN
-F 1 "20pF" H 2250 7250 50  0000 L CNN
+F 1 "?pF" H 2300 7250 50  0000 L CNN
 F 2 "Capacitor_SMD:C_0603_1608Metric" H 2200 7150 50  0001 C CNN
 F 3 "~" H 2200 7150 50  0001 C CNN
@@
 F 0 "Y2" H 5550 3825 50  0000 C CNN
 F 1 "32k 20ppm" H 5550 3734 50  0000 C CNN
-F 2 "" H 5550 3600 50  0001 C CNN
+F 2 "Crystal:Crystal_SMD_3215-2Pin_3.2x1.5mm" H 5550 3600 50  0001 C CNN
 F 3 "~" H 5550 3600 50  0001 C CNN
 	1    5550 3600
@@
 P 5750 3750
 F 0 "C16" H 5850 3750 50  0000 L CNN
-F 1 "20pF" H 5800 3650 50  0000 L CNN
+F 1 "?pF" H 5850 3650 50  0000 L CNN
 F 2 "Capacitor_SMD:C_0603_1608Metric" H 5750 3750 50  0001 C CNN
 F 3 "~" H 5750 3750 50  0001 C CNN
@@
 U 1 1 5F7EEBFB
 P 5350 3750
-F 0 "C15" H 5150 3750 50  0000 L CNN
-F 1 "20pF" H 5100 3650 50  0000 L CNN
+F 0 "C15" H 5100 3750 50  0000 L CNN
+F 1 "?pF" H 5100 3650 50  0000 L CNN
 F 2 "Capacitor_SMD:C_0603_1608Metric" H 5350 3750 50  0001 C CNN
 F 3 "~" H 5350 3750 50  0001 C CNN
@@
 	0    1    1    0
 $EndComp
-NoConn ~ 9450 1950
-NoConn ~ 9450 1850
 Text GLabel 9350 1750 0    50   Input ~ 0
 SVP
@@
 Wire Wire Line
 	950  7250 1250 7250
+$Comp
+L power:+3V3 #PWR010
+U 1 1 5F90819A
+P 9050 1750
+F 0 "#PWR010" H 9050 1600 50  0001 C CNN
+F 1 "+3V3" H 9050 1900 50  0000 C CNN
+F 2 "" H 9050 1750 50  0001 C CNN
+F 3 "" H 9050 1750 50  0001 C CNN
+	1    9050 1750
+	1    0    0    -1
+$EndComp
+$Comp
+L power:GND #PWR09
+U 1 1 5F908A0D
+P 9000 1950
+F 0 "#PWR09" H 9000 1700 50  0001 C CNN
+F 1 "GND" V 9000 1750 50  0000 C CNN
+F 2 "" H 9000 1950 50  0001 C CNN
+F 3 "" H 9000 1950 50  0001 C CNN
+	1    9000 1950
+	0    1    1    0
+$EndComp
+Wire Wire Line
+	9050 1750 9050 1850
+Wire Wire Line
+	9050 1850 9450 1850
+Wire Wire Line
+	9000 1950 9450 1950
 $EndSCHEMATC

Commit message: Schematic update
Parts:
- added J4: Conn_01x20_Male, Connector_PinHeader_2.54mm:PinHeader_1x20_P2.54mm_Vertical, symbol Connector:Conn_01x20_Male
Changed lines of the file:
@@
 U 1 1 5F795AE0
 P 4500 5850
-F 0 "R12" V 4400 5700 50  0000 L CNN
-F 1 "0R" V 4400 5850 50  0000 L CNN
+F 0 "R12" V 4400 5650 50  0000 L CNN
+F 1 "0R" V 4400 5900 50  0000 L CNN
 F 2 "Resistor_SMD:R_0603_1608Metric" V 4540 5840 50  0001 C CNN
 F 3 "~" H 4500 5850 50  0001 C CNN
@@
 P 4500 5950
 F 0 "R13" V 4400 6000 50  0000 L CNN
-F 1 "0R" V 4400 5850 50  0000 L CNN
+F 1 "0R" V 4400 5800 50  0000 L CNN
 F 2 "Resistor_SMD:R_0603_1608Metric" V 4540 5940 50  0001 C CNN
 F 3 "~" H 4500 5950 50  0001 C CNN
@@
 Wire Wire Line
 	9000 1950 9450 1950
+$Comp
+L Connector:Conn_01x20_Male J4
+U 1 1 5F63B944
+P -950 6050
+F 0 "J4" H -842 7131 50  0000 C CNN
+F 1 "Conn_01x20_Male" H -842 7040 50  0000 C CNN
+F 2 "Connector_PinHeader_2.54mm:PinHeader_1x20_P2.54mm_Vertical" H -950 6050 50  0001 C CNN
+F 3 "~" H -950 6050 50  0001 C CNN
+	1    -950 6050
+	1    0    0    -1
+$EndComp
 $EndSCHEMATC
